File: Loadstar_TKL.kicad_pcb (KiCad board)
At the start: 2 copper layers, 304.8 x 96.8 mm, 143 parts, among them J1 USB4085-GF-A_REVB, SW1 SW_Push, SW10 SW_Push, SW11 SW_Push, SW12 SW_Push, SW13 SW_Push, SW14 SW_Push, SW15 SW_Push, SW16 SW_Push, SW17 SW_Push, SW18 SW_Push, SW19 SW_Push, SW2 SW_Push, SW20 SW_Push, SW21 SW_Push, SW22 SW_Push, SW23 SW_Push, SW24 SW_Push, SW25 SW_Push, SW26 SW_Push, SW27 SW_Push, SW28 SW_Push, SW29 SW_Push, SW3 SW_Push, SW30 SW_Push, SW31 SW_Push, SW32 SW_Push, SW33 SW_Push, SW34 SW_Push, SW35 SW_Push, SW36 SW_Push, SW37 SW_Push, SW38 SW_Push, SW39 SW_Push, SW4 SW_Push, SW40 SW_Push, SW41 SW_Push, SW42 SW_Push, SW43 SW_Push, SW44 SW_Push, SW45 SW_Push, SW46 SW_Push, SW47 SW_Push, SW48 SW_Push, SW49 SW_Push, SW5 SW_Push, SW50 SW_Push, SW51 SW_Push, SW52 SW_Push, SW53 SW_Push, SW54 SW_Push, SW55 SW_Push, SW56 SW_Push, SW57 SW_Push, SW58 SW_Push, SW59 SW_Push, SW6 SW_Push, SW60 SW_Push, SW61 SW_Push, SW62 SW_Push, SW63 SW_Push, SW64 SW_Push, SW65 SW_Push, SW66 SW_Push, SW67 SW_Push, SW68 SW_Push, SW7 SW_Push, SW8 SW_Push, SW9 SW_Push, U2 ATMEGA32U4RC-MUR

Commit message: progress update
Parts:
- added LED1: 4960, Snapeda:4960_ADA, F.Cu at (33.0, 62.5)
- added LED10: 4960, Snapeda:4960_ADA, F.Cu at (223.5, 62.5)
- added LED11: 4960, Snapeda:4960_ADA, F.Cu at (242.5, 62.5)
- added LED12: 4960, Snapeda:4960_ADA, F.Cu at (261.8, 62.5)
- added LED13: 4960, Snapeda:4960_ADA, F.Cu at (280.6, 62.2)
- added LED14: 4960, Snapeda:4960_ADA, F.Cu at (299.7, 62.5)
- added LED15: 4960, Snapeda:4960_ADA, F.Cu at (319.0, 62.2)
- added LED16: 4960, Snapeda:4960_ADA, F.Cu at (33.0, 81.5)
- added LED17: 4960, Snapeda:4960_ADA, F.Cu at (302.6, 36.6)
- added LED18: 4960, Snapeda:4960_ADA, F.Cu at (308.6, 36.6)
- added LED19: 4960, Snapeda:4960_ADA, F.Cu at (314.7, 36.6)
- added LED2: 4960, Snapeda:4960_ADA, F.Cu at (61.7, 62.5)
- added LED20: 4960, Snapeda:4960_ADA, F.Cu at (320.7, 36.6)
- added LED21: 4960, Snapeda:4960_ADA, F.Cu at (326.7, 36.6)
- added LED22: 4960, Snapeda:4960_ADA, F.Cu at (272.5, 28.2)
- added LED23: 4960, Snapeda:4960_ADA, F.Cu at (278.6, 28.2)
- added LED24: 4960, Snapeda:4960_ADA, F.Cu at (284.6, 28.2)
- added LED25: 4960, Snapeda:4960_ADA, F.Cu at (290.6, 28.2)
- added LED26: 4960, Snapeda:4960_ADA, F.Cu at (296.6, 28.2)
- added LED27: 4960, Snapeda:4960_ADA, F.Cu at (302.6, 28.2)
- added LED28: 4960, Snapeda:4960_ADA, F.Cu at (308.6, 28.2)
- added LED29: 4960, Snapeda:4960_ADA, F.Cu at (314.7, 28.2)
- added LED3: 4960, Snapeda:4960_ADA, F.Cu at (90.1, 62.5)
- added LED30: 4960, Snapeda:4960_ADA, F.Cu at (320.7, 28.2)
- added LED31: 4960, Snapeda:4960_ADA, F.Cu at (326.7, 28.2)
- added LED32: 4960, Snapeda:4960_ADA, F.Cu at (272.5, 19.7)
- added LED33: 4960, Snapeda:4960_ADA, F.Cu at (278.6, 19.7)
- added LED34: 4960, Snapeda:4960_ADA, F.Cu at (284.6, 19.7)
- added LED35: 4960, Snapeda:4960_ADA, F.Cu at (290.6, 19.7)
- added LED36: 4960, Snapeda:4960_ADA, F.Cu at (296.6, 19.7)
- added LED37: 4960, Snapeda:4960_ADA, F.Cu at (302.6, 19.7)
- added LED38: 4960, Snapeda:4960_ADA, F.Cu at (308.6, 19.7)
- added LED39: 4960, Snapeda:4960_ADA, F.Cu at (314.7, 19.7)
- added LED4: 4960, Snapeda:4960_ADA, F.Cu at (109.2, 62.5)
- added LED40: 4960, Snapeda:4960_ADA, F.Cu at (320.7, 19.7)
- added LED41: 4960, Snapeda:4960_ADA, F.Cu at (326.7, 19.7)
- added LED42: 4960, Snapeda:4960_ADA, F.Cu at (272.5, 11.2)
- added LED43: 4960, Snapeda:4960_ADA, F.Cu at (278.6, 11.2)
- added LED44: 4960, Snapeda:4960_ADA, F.Cu at (284.6, 11.2)
- added LED45: 4960, Snapeda:4960_ADA, F.Cu at (290.6, 11.2)
- added LED46: 4960, Snapeda:4960_ADA, F.Cu at (296.6, 11.2)
- added LED47: 4960, Snapeda:4960_ADA, F.Cu at (302.6, 11.2)
- added LED48: 4960, Snapeda:4960_ADA, F.Cu at (308.6, 11.2)
- added LED49: 4960, Snapeda:4960_ADA, F.Cu at (314.7, 11.2)
- added LED5: 4960, Snapeda:4960_ADA, F.Cu at (128.5, 62.5)
- added LED50: 4960, Snapeda:4960_ADA, F.Cu at (320.7, 11.2)
- added LED51: 4960, Snapeda:4960_ADA, F.Cu at (326.7, 11.2)
- added LED52: 4960, Snapeda:4960_ADA, F.Cu at (272.5, 2.75)
- added LED53: 4960, Snapeda:4960_ADA, F.Cu at (278.6, 2.75)
- added LED54: 4960, Snapeda:4960_ADA, F.Cu at (284.6, 2.75)
- added LED55: 4960, Snapeda:4960_ADA, F.Cu at (290.6, 2.75)
- added LED56: 4960, Snapeda:4960_ADA, F.Cu at (296.6, 2.75)
- added LED57: 4960, Snapeda:4960_ADA, F.Cu at (302.6, 2.75)
- added LED58: 4960, Snapeda:4960_ADA, F.Cu at (308.6, 2.75)
- added LED59: 4960, Snapeda:4960_ADA, F.Cu at (314.7, 2.75)
- added LED6: 4960, Snapeda:4960_ADA, F.Cu at (147.3, 62.5)
- added LED60: 4960, Snapeda:4960_ADA, F.Cu at (320.7, 2.75)
- added LED61: 4960, Snapeda:4960_ADA, F.Cu at (326.7, 2.75)
- added LED62: 4960, Snapeda:4960_ADA, F.Cu at (272.5, -5.71)
- added LED63: 4960, Snapeda:4960_ADA, F.Cu at (278.6, -5.71)
- added LED64: 4960, Snapeda:4960_ADA, F.Cu at (284.6, -5.71)
- added LED65: 4960, Snapeda:4960_ADA, F.Cu at (290.6, -5.71)
- added LED66: 4960, Snapeda:4960_ADA, F.Cu at (296.6, -5.71)
- added LED67: 4960, Snapeda:4960_ADA, F.Cu at (302.6, -5.71)
- added LED68: 4960, Snapeda:4960_ADA, F.Cu at (308.6, -5.71)
- added LED7: 4960, Snapeda:4960_ADA, F.Cu at (166.3, 62.5)
- added LED8: 4960, Snapeda:4960_ADA, F.Cu at (185.4, 62.5)
- added LED9: 4960, Snapeda:4960_ADA, F.Cu at (204.7, 62.5)
- moved U2 88.3 mm to (227.6, 132.1), turned to -45 degrees
- moved D15 11.0 mm to (36.8, 50.3), turned to -90 degrees
- moved D17 10.9 mm to (317.7, 69.1), turned to -90 degrees
- moved D18 10.9 mm to (294.0, 69.1), turned to -90 degrees
- moved D19 10.9 mm to (274.9, 69.1), turned to -90 degrees
- moved D20 10.9 mm to (255.9, 69.1), turned to -90 degrees
- moved D21 10.9 mm to (236.8, 69.1), turned to -90 degrees
- moved D22 10.9 mm to (217.8, 69.1), turned to -90 degrees
- moved D23 10.9 mm to (198.7, 69.1), turned to -90 degrees
- moved D24 10.9 mm to (179.7, 69.1), turned to -90 degrees
- moved D25 10.9 mm to (160.6, 69.1), turned to -90 degrees
- moved D26 10.9 mm to (141.6, 69.1), turned to -90 degrees
- moved D27 10.9 mm to (122.5, 69.1), turned to -90 degrees
- moved D28 10.9 mm to (103.5, 69.1), turned to -90 degrees
- moved D29 10.9 mm to (84.4, 69.1), turned to -90 degrees
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Connections:
- D16 pad 1: row0 -> row2
- D32 pad 1: row1 -> row3
- J1 pad A1: unconnected-(J1-GND-PadA1) -> GND
- J1 pad A12: unconnected-(J1-GND__1-PadA12) -> GND
- J1 pad A4: unconnected-(J1-VBUS-PadA4) -> +5V
- J1 pad A6: unconnected-(J1-DP1-PadA6) -> Net-(J1-DP1)
- J1 pad A7: unconnected-(J1-DN1-PadA7) -> Net-(J1-DN1)
- J1 pad A9: unconnected-(J1-VBUS__1-PadA9) -> +5V
- J1 pad B1: unconnected-(J1-GND__2-PadB1) -> GND
- J1 pad B12: unconnected-(J1-GND__3-PadB12) -> GND
- J1 pad B4: unconnected-(J1-VBUS__2-PadB4) -> +5V
- J1 pad B6: unconnected-(J1-DP2-PadB6) -> Net-(J1-DP1)
- J1 pad B7: unconnected-(J1-DN2-PadB7) -> Net-(J1-DN1)
- J1 pad B9: unconnected-(J1-VBUS__3-PadB9) -> +5V
- J1 pad S1: unconnected-(J1-SHELL-PadS1) -> GND
- J1 pad S2: unconnected-(J1-SHELL__1-PadS2) -> GND
- J1 pad S3: unconnected-(J1-SHELL__2-PadS3) -> GND
- J1 pad S4: unconnected-(J1-SHELL__3-PadS4) -> GND
- SW15 pad 1: col15 -> col16
- SW31 pad 1: col15 -> col16
- U2 pad 14: unconnected-(U2-VCC-Pad14) -> +5V
- U2 pad 15: unconnected-(U2-GND-Pad15) -> GND
- U2 pad 23: unconnected-(U2-GND-Pad23) -> GND
- U2 pad 24: unconnected-(U2-AVCC-Pad24) -> +5V
- U2 pad 3: unconnected-(U2-D--Pad3) -> D-
- U2 pad 34: unconnected-(U2-VCC-Pad34) -> +5V
- U2 pad 35: unconnected-(U2-GND-Pad35) -> GND
- U2 pad 4: unconnected-(U2-D+-Pad4) -> D+
- U2 pad 43: unconnected-(U2-GND-Pad43) -> GND

Commit message: wip update
Parts:
- removed the LED58 at (308.6, 2.75)
- added D1: 1N4007, Diode_SMD:D_SOD-123, F.Cu at (328.3, 50.0)
- added D32: 1N4007, Diode_SMD:D_SOD-123, F.Cu at (327.1, 76.2)
- added D47: 1N4007, Diode_SMD:D_SOD-123, F.Cu at (327.1, 95.2)
- added D62: 1N4007, Diode_SMD:D_SOD-123, F.Cu at (327.1, 114.3)
- added D73: 1N4007, Diode_SMD:D_SOD-123, F.Cu at (327.1, 133.3)
- added LED16: 4960, Snapeda:4960_ADA, F.Cu at (33.0, 71.0)
- added LED32: 4960, Snapeda:4960_ADA, F.Cu at (33.0, 90.0)
- added LED34: 4960, Snapeda:4960_ADA, F.Cu at (94.9, 90.0)
- added LED47: 4960, Snapeda:4960_ADA, F.Cu at (33.0, 109.1)
- added LED63: 4960, Snapeda:4960_ADA, F.Cu at (33.0, 128.1)
- added REF**: Stabilizer_Cherry_MX_2.00u, PCM_Mounting_Keyboard_Stabilizer:Stabilizer_Cherry_MX_2.00u, B.Cu at (61.6, 57.1)
- added REF**: Stabilizer_Cherry_MX_6.25u, PCM_Mounting_Keyboard_Stabilizer:Stabilizer_Cherry_MX_6.25u, B.Cu at (197.3, 133.3)
- added REF**: Stabilizer_Cherry_MX_2.00u, PCM_Mounting_Keyboard_Stabilizer:Stabilizer_Cherry_MX_2.00u, B.Cu at (63.9, 95.2)
- added REF**: Stabilizer_Cherry_MX_2.00u, PCM_Mounting_Keyboard_Stabilizer:Stabilizer_Cherry_MX_2.00u, B.Cu at (306.8, 114.3)
- added SW16: RotaryEncoder_Switch, Rotary_Encoder:RotaryEncoder_Alps_EC11E-Switch_Vertical_H20mm, B.Cu at (340.3, 64.7)
- added SW17: SW_Push, PCM_Switch_Keyboard_Hotswap_Kailh:SW_Hotswap_Kailh_MX_Plated_1.00u, B.Cu at (337.8, 76.2)
- added SW33: SW_Push, PCM_Switch_Keyboard_Hotswap_Kailh:SW_Hotswap_Kailh_MX_Plated_1.00u, B.Cu at (337.8, 95.2)
- added SW48: SW_Push, PCM_Switch_Keyboard_Hotswap_Kailh:SW_Hotswap_Kailh_MX_Plated_1.00u, B.Cu at (337.8, 114.3)
- added SW63: SW_Push, PCM_Switch_Keyboard_Hotswap_Kailh:SW_Hotswap_Kailh_MX_Plated_1.00u, B.Cu at (337.8, 133.3)
- J1: value USB4085-GF-A_REVB -> USB-C
- SW1, SW10, SW11, SW12, SW13, SW15, SW2, SW3, SW4, SW5, SW6, SW7, SW8, SW9: footprint Button_Switch_Keyboard:SW_Cherry_MX_1.00u_PCB -> PCM_Switch_Keyboard_Hotswap_Kailh:SW_Hotswap_Kailh_MX_Plated_1.00u
- SW14: footprint Button_Switch_Keyboard:SW_Cherry_MX_2.00u_PCB -> PCM_Switch_Keyboard_Hotswap_Kailh:SW_Hotswap_Kailh_MX_Plated_2.00u
- SW18: renamed from SW17; footprint Button_Switch_Keyboard:SW_Cherry_MX_1.50u_PCB -> PCM_Switch_Keyboard_Hotswap_Kailh:SW_Hotswap_Kailh_MX_Plated_1.50u
- SW19: renamed from SW18; footprint Button_Switch_Keyboard:SW_Cherry_MX_1.00u_PCB -> PCM_Switch_Keyboard_Hotswap_Kailh:SW_Hotswap_Kailh_MX_Plated_1.00u
- SW20: renamed from SW19; footprint Button_Switch_Keyboard:SW_Cherry_MX_1.00u_PCB -> PCM_Switch_Keyboard_Hotswap_Kailh:SW_Hotswap_Kailh_MX_Plated_1.00u
- SW21: renamed from SW20; footprint Button_Switch_Keyboard:SW_Cherry_MX_1.00u_PCB -> PCM_Switch_Keyboard_Hotswap_Kailh:SW_Hotswap_Kailh_MX_Plated_1.00u
- SW22: renamed from SW21; footprint Button_Switch_Keyboard:SW_Cherry_MX_1.00u_PCB -> PCM_Switch_Keyboard_Hotswap_Kailh:SW_Hotswap_Kailh_MX_Plated_1.00u
- SW23: renamed from SW22; footprint Button_Switch_Keyboard:SW_Cherry_MX_1.00u_PCB -> PCM_Switch_Keyboard_Hotswap_Kailh:SW_Hotswap_Kailh_MX_Plated_1.00u
- SW24: renamed from SW23; footprint Button_Switch_Keyboard:SW_Cherry_MX_1.00u_PCB -> PCM_Switch_Keyboard_Hotswap_Kailh:SW_Hotswap_Kailh_MX_Plated_1.00u
- SW25: renamed from SW24; footprint Button_Switch_Keyboard:SW_Cherry_MX_1.00u_PCB -> PCM_Switch_Keyboard_Hotswap_Kailh:SW_Hotswap_Kailh_MX_Plated_1.00u
- SW26: renamed from SW25; footprint Button_Switch_Keyboard:SW_Cherry_MX_1.00u_PCB -> PCM_Switch_Keyboard_Hotswap_Kailh:SW_Hotswap_Kailh_MX_Plated_1.00u
- SW27: renamed from SW26; footprint Button_Switch_Keyboard:SW_Cherry_MX_1.00u_PCB -> PCM_Switch_Keyboard_Hotswap_Kailh:SW_Hotswap_Kailh_MX_Plated_1.00u
- SW28: renamed from SW27; footprint Button_Switch_Keyboard:SW_Cherry_MX_1.00u_PCB -> PCM_Switch_Keyboard_Hotswap_Kailh:SW_Hotswap_Kailh_MX_Plated_1.00u
- SW29: renamed from SW28; footprint Button_Switch_Keyboard:SW_Cherry_MX_1.00u_PCB -> PCM_Switch_Keyboard_Hotswap_Kailh:SW_Hotswap_Kailh_MX_Plated_1.00u
- SW30: renamed from SW29; footprint Button_Switch_Keyboard:SW_Cherry_MX_1.00u_PCB -> PCM_Switch_Keyboard_Hotswap_Kailh:SW_Hotswap_Kailh_MX_Plated_1.00u
- SW31: renamed from SW30; footprint Button_Switch_Keyboard:SW_Cherry_MX_1.50u_PCB -> PCM_Switch_Keyboard_Hotswap_Kailh:SW_Hotswap_Kailh_MX_Plated_1.50u
- SW32: renamed from SW31; footprint Button_Switch_Keyboard:SW_Cherry_MX_1.00u_PCB -> PCM_Switch_Keyboard_Hotswap_Kailh:SW_Hotswap_Kailh_MX_Plated_1.00u
- SW34: renamed from SW33; footprint Button_Switch_Keyboard:SW_Cherry_MX_1.75u_PCB -> PCM_Switch_Keyboard_Hotswap_Kailh:SW_Hotswap_Kailh_MX_Plated_1.75u
- SW35: renamed from SW34; footprint Button_Switch_Keyboard:SW_Cherry_MX_1.00u_PCB -> PCM_Switch_Keyboard_Hotswap_Kailh:SW_Hotswap_Kailh_MX_Plated_1.00u
- SW36: renamed from SW35; footprint Button_Switch_Keyboard:SW_Cherry_MX_1.00u_PCB -> PCM_Switch_Keyboard_Hotswap_Kailh:SW_Hotswap_Kailh_MX_Plated_1.00u
- SW37: renamed from SW36; footprint Button_Switch_Keyboard:SW_Cherry_MX_1.00u_PCB -> PCM_Switch_Keyboard_Hotswap_Kailh:SW_Hotswap_Kailh_MX_Plated_1.00u
- SW38: renamed from SW37; footprint Button_Switch_Keyboard:SW_Cherry_MX_1.00u_PCB -> PCM_Switch_Keyboard_Hotswap_Kailh:SW_Hotswap_Kailh_MX_Plated_1.00u
- SW39: renamed from SW38; footprint Button_Switch_Keyboard:SW_Cherry_MX_1.00u_PCB -> PCM_Switch_Keyboard_Hotswap_Kailh:SW_Hotswap_Kailh_MX_Plated_1.00u
- SW40: renamed from SW39; footprint Button_Switch_Keyboard:SW_Cherry_MX_1.00u_PCB -> PCM_Switch_Keyboard_Hotswap_Kailh:SW_Hotswap_Kailh_MX_Plated_1.00u
- SW41: renamed from SW40; footprint Button_Switch_Keyboard:SW_Cherry_MX_1.00u_PCB -> PCM_Switch_Keyboard_Hotswap_Kailh:SW_Hotswap_Kailh_MX_Plated_1.00u
- SW42: renamed from SW41; footprint Button_Switch_Keyboard:SW_Cherry_MX_1.00u_PCB -> PCM_Switch_Keyboard_Hotswap_Kailh:SW_Hotswap_Kailh_MX_Plated_1.00u
- SW43: renamed from SW42; footprint Button_Switch_Keyboard:SW_Cherry_MX_1.00u_PCB -> PCM_Switch_Keyboard_Hotswap_Kailh:SW_Hotswap_Kailh_MX_Plated_1.00u
- SW44: renamed from SW43; footprint Button_Switch_Keyboard:SW_Cherry_MX_1.00u_PCB -> PCM_Switch_Keyboard_Hotswap_Kailh:SW_Hotswap_Kailh_MX_Plated_1.00u
- SW45: renamed from SW44; footprint Button_Switch_Keyboard:SW_Cherry_MX_1.00u_PCB -> PCM_Switch_Keyboard_Hotswap_Kailh:SW_Hotswap_Kailh_MX_Plated_1.00u
- SW46: renamed from SW45; footprint Button_Switch_Keyboard:SW_Cherry_MX_2.25u_PCB -> PCM_Switch_Keyboard_Hotswap_Kailh:SW_Hotswap_Kailh_MX_Plated_2.25u
- SW47: renamed from SW16; footprint Button_Switch_Keyboard:SW_Cherry_MX_1.00u_PCB -> PCM_Switch_Keyboard_Hotswap_Kailh:SW_Hotswap_Kailh_MX_Plated_1.00u
- SW49: renamed from SW46; footprint Button_Switch_Keyboard:SW_Cherry_MX_2.25u_PCB -> PCM_Switch_Keyboard_Hotswap_Kailh:SW_Hotswap_Kailh_MX_Plated_2.25u
- SW50: renamed from SW47; footprint Button_Switch_Keyboard:SW_Cherry_MX_1.00u_PCB -> PCM_Switch_Keyboard_Hotswap_Kailh:SW_Hotswap_Kailh_MX_Plated_1.00u
- SW51: renamed from SW48; footprint Button_Switch_Keyboard:SW_Cherry_MX_1.00u_PCB -> PCM_Switch_Keyboard_Hotswap_Kailh:SW_Hotswap_Kailh_MX_Plated_1.00u
- SW52: renamed from SW49; footprint Button_Switch_Keyboard:SW_Cherry_MX_1.00u_PCB -> PCM_Switch_Keyboard_Hotswap_Kailh:SW_Hotswap_Kailh_MX_Plated_1.00u
- SW53: renamed from SW50; footprint Button_Switch_Keyboard:SW_Cherry_MX_1.00u_PCB -> PCM_Switch_Keyboard_Hotswap_Kailh:SW_Hotswap_Kailh_MX_Plated_1.00u
- SW54: renamed from SW51; footprint Button_Switch_Keyboard:SW_Cherry_MX_1.00u_PCB -> PCM_Switch_Keyboard_Hotswap_Kailh:SW_Hotswap_Kailh_MX_Plated_1.00u
- SW55: renamed from SW52; footprint Button_Switch_Keyboard:SW_Cherry_MX_1.00u_PCB -> PCM_Switch_Keyboard_Hotswap_Kailh:SW_Hotswap_Kailh_MX_Plated_1.00u
- SW56: renamed from SW53; footprint Button_Switch_Keyboard:SW_Cherry_MX_1.00u_PCB -> PCM_Switch_Keyboard_Hotswap_Kailh:SW_Hotswap_Kailh_MX_Plated_1.00u
- SW57: renamed from SW54; footprint Button_Switch_Keyboard:SW_Cherry_MX_1.00u_PCB -> PCM_Switch_Keyboard_Hotswap_Kailh:SW_Hotswap_Kailh_MX_Plated_1.00u
- SW58: renamed from SW55; footprint Button_Switch_Keyboard:SW_Cherry_MX_1.00u_PCB -> PCM_Switch_Keyboard_Hotswap_Kailh:SW_Hotswap_Kailh_MX_Plated_1.00u
- SW59: renamed from SW56; footprint Button_Switch_Keyboard:SW_Cherry_MX_1.00u_PCB -> PCM_Switch_Keyboard_Hotswap_Kailh:SW_Hotswap_Kailh_MX_Plated_1.00u
- SW60: renamed from SW57; footprint Button_Switch_Keyboard:SW_Cherry_MX_1.75u_PCB -> PCM_Switch_Keyboard_Hotswap_Kailh:SW_Hotswap_Kailh_MX_Plated_1.75u
- SW61: renamed from SW58; footprint Button_Switch_Keyboard:SW_Cherry_MX_1.00u_PCB -> PCM_Switch_Keyboard_Hotswap_Kailh:SW_Hotswap_Kailh_MX_Plated_1.00u
- SW62: renamed from SW32; footprint Button_Switch_Keyboard:SW_Cherry_MX_1.00u_PCB -> PCM_Switch_Keyboard_Hotswap_Kailh:SW_Hotswap_Kailh_MX_Plated_1.00u
- SW64: renamed from SW59; footprint Button_Switch_Keyboard:SW_Cherry_MX_1.25u_PCB -> PCM_Switch_Keyboard_Hotswap_Kailh:SW_Hotswap_Kailh_MX_Plated_1.25u
- SW65: renamed from SW60; footprint Button_Switch_Keyboard:SW_Cherry_MX_1.25u_PCB -> PCM_Switch_Keyboard_Hotswap_Kailh:SW_Hotswap_Kailh_MX_Plated_1.25u
- SW66: renamed from SW61; footprint Button_Switch_Keyboard:SW_Cherry_MX_1.25u_PCB -> PCM_Switch_Keyboard_Hotswap_Kailh:SW_Hotswap_Kailh_MX_Plated_1.25u
- SW67: renamed from SW62; footprint Button_Switch_Keyboard:SW_Cherry_MX_6.25u_PCB -> PCM_Switch_Keyboard_Hotswap_Kailh:SW_Hotswap_Kailh_MX_Plated_6.25u
- SW68: renamed from SW63; footprint Button_Switch_Keyboard:SW_Cherry_MX_1.00u_PCB -> PCM_Switch_Keyboard_Hotswap_Kailh:SW_Hotswap_Kailh_MX_Plated_1.00u
- SW69: renamed from SW64; footprint Button_Switch_Keyboard:SW_Cherry_MX_1.00u_PCB -> PCM_Switch_Keyboard_Hotswap_Kailh:SW_Hotswap_Kailh_MX_Plated_1.00u
- SW70: renamed from SW65; footprint Button_Switch_Keyboard:SW_Cherry_MX_1.00u_PCB -> PCM_Switch_Keyboard_Hotswap_Kailh:SW_Hotswap_Kailh_MX_Plated_1.00u
- SW71: renamed from SW66; footprint Button_Switch_Keyboard:SW_Cherry_MX_1.00u_PCB -> PCM_Switch_Keyboard_Hotswap_Kailh:SW_Hotswap_Kailh_MX_Plated_1.00u
- SW72: renamed from SW67; footprint Button_Switch_Keyboard:SW_Cherry_MX_1.00u_PCB -> PCM_Switch_Keyboard_Hotswap_Kailh:SW_Hotswap_Kailh_MX_Plated_1.00u
- SW73: renamed from SW68; footprint Button_Switch_Keyboard:SW_Cherry_MX_1.00u_PCB -> PCM_Switch_Keyboard_Hotswap_Kailh:SW_Hotswap_Kailh_MX_Plated_1.00u
- moved LED64 291.0 mm to (52.0, 128.1), turned to 0 degrees
- moved LED62 279.3 mm to (71.1, 128.1), turned to 0 degrees
- moved LED33 269.9 mm to (63.9, 90.0), turned to 0 degrees
- moved LED65 267.7 mm to (90.1, 128.1), turned to 0 degrees
- moved LED48 252.3 mm to (52.0, 109.1), turned to 0 degrees
- moved J1 246.4 mm to (81.7, 45.0), turned to 180 degrees
- moved LED49 233.8 mm to (78.2, 109.1), turned to 0 degrees
- moved LED18 224.7 mm to (80.6, 71.0), turned to 0 degrees
- moved LED50 215.7 mm to (104.4, 109.1), turned to 0 degrees
- moved LED19 211.8 mm to (99.7, 71.0), turned to 0 degrees
- moved LED66 211.2 mm to (109.2, 128.1), turned to 0 degrees
- moved LED51 204.1 mm to (123.5, 109.1), turned to 0 degrees
- moved LED67 201.3 mm to (128.2, 128.1), turned to 0 degrees
- moved LED20 198.9 mm to (118.7, 71.0), turned to 0 degrees
- moved LED56 192.8 mm to (142.5, 109.1), turned to 0 degrees
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- renumbered D7 to D10, D6 to D11, D5 to D12, D4 to D13, D3 to D14, D2 to D15, D1 to D16, D31 to D17, D30 to D18, D29 to D19, D15 to D2, D28 to D20, D27 to D21, D26 to D22, D25 to D23, D23 to D25, D22 to D26, D21 to D27, D20 to D28, D19 to D29, D14 to D3, D18 to D30, D17 to D31, D16 to D33, D45 to D34, D44 to D35, D43 to D36, D42 to D37, D41 to D38, D40 to D39, D13 to D4, D39 to D40, D38 to D41, D37 to D42, D36 to D43, D35 to D44, D34 to D45, D33 to D46, D32 to D48, D58 to D49, D12 to D5, D57 to D50, D56 to D51, D55 to D52, D54 to D53, D53 to D54, D52 to D55, D51 to D56, D50 to D57, D49 to D58, D48 to D59, D11 to D6, D47 to D60, D46 to D61, D68 to D63, D67 to D64, D66 to D65, D65 to D66, D64 to D67, D63 to D68, D62 to D69, D10 to D7, D61 to D70, D60 to D71, D59 to D72, D9 to D8, D8 to D9, LED16 to LED17, LED17 to LED18, LED18 to LED19, LED19 to LED20, LED20 to LED21, LED21 to LED22, LED22 to LED23, LED23 to LED24, LED24 to LED25, LED25 to LED26, LED26 to LED27, LED27 to LED28, LED28 to LED29, LED29 to LED30, LED30 to LED31, LED31 to LED33, LED32 to LED35, LED33 to LED36, LED34 to LED37, LED35 to LED38, LED36 to LED39, LED37 to LED40, LED38 to LED41, LED39 to LED42, LED40 to LED43, LED41 to LED44, LED42 to LED45, LED43 to LED46, LED44 to LED48, LED45 to LED49, LED46 to LED50, LED47 to LED51, LED54 to LED53, LED55 to LED54, LED56 to LED55, LED48 to LED56, LED49 to LED57, LED50 to LED58, LED51 to LED59, LED53 to LED60, LED57 to LED61, LED60 to LED62, LED59 to LED64, LED61 to LED65, LED62 to LED66, LED63 to LED67, LED64 to LED68, LED65 to LED69, LED66 to LED70, LED67 to LED71, LED68 to LED72, U2 to U1
Connections:
- J1 pad A4: +5V -> Net-(J1-VBUS)
- J1 pad A5: unconnected-(J1-CC1-PadA5) -> Net-(J1-CC1)
- J1 pad A9: +5V -> Net-(J1-VBUS)
- J1 pad B4: +5V -> Net-(J1-VBUS)
- J1 pad B5: unconnected-(J1-CC2-PadB5) -> Net-(J1-CC2)
- J1 pad B9: +5V -> Net-(J1-VBUS)
- LED1 pad 2: unconnected-(LED1-DOUT-Pad2) -> Net-(LED1-DOUT)
- LED17 pad 2: unconnected-(LED16-DOUT-Pad2) -> Net-(LED16-DOUT)
- LED33 pad 2: unconnected-(LED31-DOUT-Pad2) -> Net-(LED31-DOUT)
- LED35 pad 2: Net-(LED31-DIN) -> Net-(LED32-DOUT)
- LED48 pad 2: unconnected-(LED44-DOUT-Pad2) -> Net-(LED44-DOUT)
- LED64 pad 2: unconnected-(LED59-DOUT-Pad2) -> Net-(LED59-DOUT)
- SW1 pad 1: col0 -> col2
- SW10 pad 1: col10 -> col11
- SW11 pad 1: col11 -> col12
- SW12 pad 1: col12 -> col13
- SW13 pad 1: col13 -> col14
- SW14 pad 1: col14 -> col15
- SW15 pad 1: col16 -> col17
- SW18 pad 1: col0 -> col2
- SW19 pad 1: col2 -> col3
- SW2 pad 1: col2 -> col3
- SW20 pad 1: col3 -> col4
- SW21 pad 1: col4 -> col5
- SW22 pad 1: col5 -> col6
- SW23 pad 1: col6 -> col7
- SW24 pad 1: col7 -> col8
- SW25 pad 1: col8 -> col9
- SW26 pad 1: col9 -> col10
- SW27 pad 1: col10 -> col11
- SW28 pad 1: col11 -> col12
- SW29 pad 1: col12 -> col13
- SW3 pad 1: col3 -> col4
- SW30 pad 1: col13 -> col14
- SW31 pad 1: col14 -> col15
- SW32 pad 1: col16 -> col17
- SW34 pad 1: col0 -> col2
- SW35 pad 1: col2 -> col3
- SW36 pad 1: col3 -> col4
- SW37 pad 1: col4 -> col5
- SW38 pad 1: col5 -> col6
- SW39 pad 1: col6 -> col7
- SW4 pad 1: col4 -> col5
- SW40 pad 1: col7 -> col8
- SW41 pad 1: col8 -> col9
- SW42 pad 1: col9 -> col10
- SW43 pad 1: col10 -> col11
- SW44 pad 1: col11 -> col12
- SW45 pad 1: col12 -> col13
- SW46 pad 1: col14 -> col15
- SW47 pad 1: col16 -> col17
- SW49 pad 1: col0 -> col2
- SW5 pad 1: col5 -> col6
- SW50 pad 1: col3 -> col4
- SW51 pad 1: col4 -> col5
- SW52 pad 1: col5 -> col6
- SW53 pad 1: col6 -> col7
- SW54 pad 1: col7 -> col8
- SW55 pad 1: col8 -> col9
- SW56 pad 1: col9 -> col10
- SW57 pad 1: col10 -> col11
- SW58 pad 1: col11 -> col12
- SW59 pad 1: col12 -> col13
- SW6 pad 1: col6 -> col7
- SW60 pad 1: col14 -> col15
- SW61 pad 1: col15 -> col16
- SW62 pad 1: col16 -> col17
- SW64 pad 1: col0 -> col2
- SW65 pad 1: col2 -> col3
- SW66 pad 1: col3 -> col4
- SW67 pad 1: col7 -> col8
- SW68 pad 1: col11 -> col12
- SW69 pad 1: col12 -> col13
- SW7 pad 1: col7 -> col8
- SW70 pad 1: col13 -> col14
- SW71 pad 1: col14 -> col15
- SW72 pad 1: col15 -> col16
- SW73 pad 1: col16 -> col17
- SW8 pad 1: col8 -> col9
- SW9 pad 1: col9 -> col10
- U1 pad 13: unconnected-(U2-*RESET-Pad13) -> RESET
- U1 pad 16: unconnected-(U2-XTAL2-Pad16) -> Net-(U2-XTAL2)
- U1 pad 17: unconnected-(U2-XTAL1-Pad17) -> Net-(U2-XTAL1)
- U1 pad 34: +5V -> unconnected-(U2-VCC-Pad34)
- U1 pad 35: GND -> unconnected-(U2-GND-Pad35)
- U1 pad 43: GND -> unconnected-(U2-GND-Pad43)
Other:
- board size 304.8 x 96.8 mm -> 324 x 99.6 mm
