File: Loadstar_TKL.kicad_sch (KiCad schematic)
At the start: 140 parts, among them J1 USB4085-GF-A_REVB, SW1 SW_Push, SW10 SW_Push, SW11 SW_Push, SW12 SW_Push, SW13 SW_Push, SW14 SW_Push, SW15 SW_Push, SW16 SW_Push, SW17 SW_Push, SW18 SW_Push, SW19 SW_Push, SW2 SW_Push, SW20 SW_Push, SW21 SW_Push, SW22 SW_Push, SW23 SW_Push, SW24 SW_Push, SW25 SW_Push, SW26 SW_Push, SW27 SW_Push, SW28 SW_Push, SW29 SW_Push, SW3 SW_Push, SW30 SW_Push, SW31 SW_Push, SW32 SW_Push, SW33 SW_Push, SW34 SW_Push, SW35 SW_Push, SW36 SW_Push, SW37 SW_Push, SW38 SW_Push, SW39 SW_Push, SW4 SW_Push, SW40 SW_Push, SW41 SW_Push, SW42 SW_Push, SW43 SW_Push, SW44 SW_Push, SW45 SW_Push, SW46 SW_Push, SW47 SW_Push, SW48 SW_Push, SW49 SW_Push, SW5 SW_Push, SW50 SW_Push, SW51 SW_Push, SW52 SW_Push, SW53 SW_Push, SW54 SW_Push, SW55 SW_Push, SW56 SW_Push, SW57 SW_Push, SW58 SW_Push, SW59 SW_Push, SW6 SW_Push, SW60 SW_Push, SW61 SW_Push, SW62 SW_Push, SW63 SW_Push, SW64 SW_Push, SW65 SW_Push, SW66 SW_Push, SW67 SW_Push, SW68 SW_Push, SW7 SW_Push, SW8 SW_Push, SW9 SW_Push, U2 ATMEGA32U4RC-MUR

Commit message: progress update
Parts:
- added LED1, LED10, LED11, LED12, LED13, LED14, LED15, LED16, LED17, LED18, LED19, LED2, LED20, LED21, LED22, LED23, LED24, LED25, LED26, LED27, LED28, LED29, LED3, LED30, LED31, LED32, LED33, LED34, LED35, LED36, LED37, LED38, LED39, LED4, LED40, LED41, LED42, LED43, LED44, LED45, LED46, LED47, LED48, LED49, LED5, LED50, LED51, LED52, LED53, LED54, LED55, LED56, LED57, LED58, LED59, LED6, LED60, LED61, LED62, LED63, LED64, LED65, LED66, LED67, LED68, LED7, LED8, LED9: 4960, Snapeda:4960_ADA, symbol Snapeda_kicad_sym:4960
Connections:
- net +5V: now also LED1.1 (VDD), LED10.1 (VDD), LED11.1 (VDD), LED12.1 (VDD), LED13.1 (VDD), LED14.1 (VDD), LED15.1 (VDD), LED16.1 (VDD), LED17.1 (VDD), LED18.1 (VDD), LED19.1 (VDD), LED2.1 (VDD), LED20.1 (VDD), LED21.1 (VDD), LED22.1 (VDD), LED23.1 (VDD), LED24.1 (VDD), LED25.1 (VDD), LED26.1 (VDD), LED27.1 (VDD), LED28.1 (VDD), LED29.1 (VDD), LED3.1 (VDD), LED30.1 (VDD), LED31.1 (VDD), LED32.1 (VDD), LED33.1 (VDD), LED34.1 (VDD), LED35.1 (VDD), LED36.1 (VDD), LED37.1 (VDD), LED38.1 (VDD), LED39.1 (VDD), LED4.1 (VDD), LED40.1 (VDD), LED41.1 (VDD), LED42.1 (VDD), LED43.1 (VDD), LED44.1 (VDD), LED45.1 (VDD), LED46.1 (VDD), LED47.1 (VDD), LED48.1 (VDD), LED49.1 (VDD), LED5.1 (VDD), LED50.1 (VDD), LED51.1 (VDD), LED52.1 (VDD), LED53.1 (VDD), LED54.1 (VDD), LED55.1 (VDD), LED56.1 (VDD), LED57.1 (VDD), LED58.1 (VDD), LED59.1 (VDD), LED6.1 (VDD), LED60.1 (VDD), LED61.1 (VDD), LED62.1 (VDD), LED63.1 (VDD), LED64.1 (VDD), LED65.1 (VDD), LED66.1 (VDD), LED67.1 (VDD), LED68.1 (VDD), LED7.1 (VDD), LED8.1 (VDD), LED9.1 (VDD)
- net GND: now also LED1.3 (GND), LED10.3 (GND), LED11.3 (GND), LED12.3 (GND), LED13.3 (GND), LED14.3 (GND), LED15.3 (GND), LED16.3 (GND), LED17.3 (GND), LED18.3 (GND), LED19.3 (GND), LED2.3 (GND), LED20.3 (GND), LED21.3 (GND), LED22.3 (GND), LED23.3 (GND), LED24.3 (GND), LED25.3 (GND), LED26.3 (GND), LED27.3 (GND), LED28.3 (GND), LED29.3 (GND), LED3.3 (GND), LED30.3 (GND), LED31.3 (GND), LED32.3 (GND), LED33.3 (GND), LED34.3 (GND), LED35.3 (GND), LED36.3 (GND), LED37.3 (GND), LED38.3 (GND), LED39.3 (GND), LED4.3 (GND), LED40.3 (GND), LED41.3 (GND), LED42.3 (GND), LED43.3 (GND), LED44.3 (GND), LED45.3 (GND), LED46.3 (GND), LED47.3 (GND), LED48.3 (GND), LED49.3 (GND), LED5.3 (GND), LED50.3 (GND), LED51.3 (GND), LED52.3 (GND), LED53.3 (GND), LED54.3 (GND), LED55.3 (GND), LED56.3 (GND), LED57.3 (GND), LED58.3 (GND), LED59.3 (GND), LED6.3 (GND), LED60.3 (GND), LED61.3 (GND), LED62.3 (GND), LED63.3 (GND), LED64.3 (GND), LED65.3 (GND), LED66.3 (GND), LED67.3 (GND), LED68.3 (GND), LED7.3 (GND), LED8.3 (GND), LED9.3 (GND)
- net col15: no longer SW15.1, SW31.1
- net col16: now also SW15.1, SW31.1
- net row0: no longer D16.1 (K)
- net row1: no longer D32.1 (K)
- net row2: now also D16.1 (K)
- net row3: now also D32.1 (K)
- new net: LED23.4 (DIN), LED24.2 (DOUT)
- new net: LED24.4 (DIN), LED25.2 (DOUT)
- new net: LED4.4 (DIN), LED5.2 (DOUT)
- new net: LED5.4 (DIN), LED6.2 (DOUT)
- new net: LED28.4 (DIN), LED29.2 (DOUT)
- new net: LED29.4 (DIN), LED30.2 (DOUT)
- new net: LED22.4 (DIN), LED23.2 (DOUT)
- new net: LED31.4 (DIN), LED32.2 (DOUT)
- new net: LED32.4 (DIN), LED33.2 (DOUT)
- new net: LED21.4 (DIN), LED22.2 (DOUT)
- new net: LED18.4 (DIN), LED19.2 (DOUT)
- new net: LED19.4 (DIN), LED20.2 (DOUT)
- new net: LED7.4 (DIN), LED8.2 (DOUT)
- new net: LED8.4 (DIN), LED9.2 (DOUT)
- new net: LED16.4 (DIN), LED17.2 (DOUT)
- new net: LED17.4 (DIN), LED18.2 (DOUT)
- new net: LED61.4 (DIN), LED62.2 (DOUT)
- new net: LED62.4 (DIN), LED63.2 (DOUT)
- new net: LED10.2 (DOUT), LED9.4 (DIN)
- new net: LED48.4 (DIN), LED49.2 (DOUT)
- new net: LED49.4 (DIN), LED50.2 (DOUT)
- new net: LED36.4 (DIN), LED37.2 (DOUT)
- new net: LED37.4 (DIN), LED38.2 (DOUT)
- new net: LED13.4 (DIN), LED14.2 (DOUT)
- new net: LED14.4 (DIN), LED15.2 (DOUT)
- new net: LED59.4 (DIN), LED60.2 (DOUT)
- new net: LED51.4 (DIN), LED52.2 (DOUT)
- new net: LED52.4 (DIN), LED53.2 (DOUT)
- new net: LED1.4 (DIN), LED2.2 (DOUT)
- new net: LED67.4 (DIN), LED68.2 (DOUT)
- new net: LED35.4 (DIN), LED36.2 (DOUT)
- new net: LED33.4 (DIN), LED34.2 (DOUT)
- new net: LED34.4 (DIN), LED35.2 (DOUT)
- new net: LED6.4 (DIN), LED7.2 (DOUT)
- new net: LED42.4 (DIN), LED43.2 (DOUT)
- new net: LED10.4 (DIN), LED11.2 (DOUT)
- new net: LED11.4 (DIN), LED12.2 (DOUT)
- new net: LED27.4 (DIN), LED28.2 (DOUT)
- new net: LED45.4 (DIN), LED46.2 (DOUT)
- new net: LED46.4 (DIN), LED47.2 (DOUT)
- new net: LED47.4 (DIN), LED48.2 (DOUT)
- new net: LED44.4 (DIN), LED45.2 (DOUT)
- new net: LED25.4 (DIN), LED26.2 (DOUT)
- new net: LED60.4 (DIN), LED61.2 (DOUT)
- new net: LED50.4 (DIN), LED51.2 (DOUT)
- new net: LED63.4 (DIN), LED64.2 (DOUT)
- new net: LED12.4 (DIN), LED13.2 (DOUT)
- new net: LED2.4 (DIN), LED3.2 (DOUT)
- new net: LED26.4 (DIN), LED27.2 (DOUT)
- new net: LED3.4 (DIN), LED4.2 (DOUT)
- new net: LED65.4 (DIN), LED66.2 (DOUT)
- new net: LED66.4 (DIN), LED67.2 (DOUT)
- new net: LED20.4 (DIN), LED21.2 (DOUT)
- new net: LED39.4 (DIN), LED40.2 (DOUT)
- new net: LED40.4 (DIN), LED41.2 (DOUT)
- new net: LED41.4 (DIN), LED42.2 (DOUT)
- new net: LED53.4 (DIN), LED54.2 (DOUT)
- new net: LED54.4 (DIN), LED55.2 (DOUT)
- new net: LED56.4 (DIN), LED57.2 (DOUT)
- new net: LED57.4 (DIN), LED58.2 (DOUT)
- new net: LED38.4 (DIN), LED39.2 (DOUT)
- new net: LED55.4 (DIN), LED56.2 (DOUT)
- new net: LED64.4 (DIN), LED65.2 (DOUT)
- new net LED_row0: LED15.4 (DIN)
- new net LED_row1: LED30.4 (DIN)
- new net LED_row2: LED43.4 (DIN)
- new net LED_row3: LED58.4 (DIN)
- new net LED_row4: LED68.4 (DIN)
Other:
- moved on the sheet: D1, D10, D11, D12, D13, D14, D17, D18, D19, D2, D20, D21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

Commit message: wip update
Parts:
- removed LED58: 4960, Snapeda:4960_ADA, symbol Snapeda_kicad_sym:4960
- added C1, C10, C11, C12, C13, C14, C15, C16, C17, C18, C19, C2, C20, C21, C22, C23, C24, C25, C26, C27, C28, C29, C30, C31, C32, C33, C34, C35, C36, C37, C38, C39, C40, C41, C42, C43, C44, C45, C46, C47, C48, C49, C5, C50, C51, C52, C53, C54, C55, C56, C57, C58, C59, C6, C60, C61, C62, C63, C64, C65, C66, C67, C68, C69, C7, C70, C71, C72, C73, C74, C75, C76, C8, C9: 0.1u, symbol Device:C
- added C3, C4: 22p, symbol Device:C
- added D1, D32, D47, D62, D73: 1N4007, Diode_SMD:D_SOD-123, symbol Diode:1N4007
- added LED16, LED32, LED34, LED47, LED63: 4960, Snapeda:4960_ADA, symbol Snapeda_kicad_sym:4960
- added R3, R4: 5.1k, symbol Device:R
- added R5: 10k, symbol Device:R
- added SW16: RotaryEncoder_Switch, Rotary_Encoder:RotaryEncoder_Alps_EC11E-Switch_Vertical_H20mm, symbol Device:RotaryEncoder_Switch
- added SW17, SW33, SW48, SW63: SW_Push, PCM_Switch_Keyboard_Hotswap_Kailh:SW_Hotswap_Kailh_MX_Plated_1.00u, symbol Switch:SW_Push
- added Y1: 16MHz, symbol Device:Crystal_Small
- J1: value USB4085-GF-A_REVB -> USB-C
- SW1, SW10, SW11, SW12, SW13, SW15, SW2, SW3, SW4, SW5, SW6, SW7, SW8, SW9: footprint Button_Switch_Keyboard:SW_Cherry_MX_1.00u_PCB -> PCM_Switch_Keyboard_Hotswap_Kailh:SW_Hotswap_Kailh_MX_Plated_1.00u
- SW14: footprint Button_Switch_Keyboard:SW_Cherry_MX_2.00u_PCB -> PCM_Switch_Keyboard_Hotswap_Kailh:SW_Hotswap_Kailh_MX_Plated_2.00u
- SW18: renamed from SW17; footprint Button_Switch_Keyboard:SW_Cherry_MX_1.50u_PCB -> PCM_Switch_Keyboard_Hotswap_Kailh:SW_Hotswap_Kailh_MX_Plated_1.50u
- SW19: renamed from SW18; footprint Button_Switch_Keyboard:SW_Cherry_MX_1.00u_PCB -> PCM_Switch_Keyboard_Hotswap_Kailh:SW_Hotswap_Kailh_MX_Plated_1.00u
- SW20: renamed from SW19; footprint Button_Switch_Keyboard:SW_Cherry_MX_1.00u_PCB -> PCM_Switch_Keyboard_Hotswap_Kailh:SW_Hotswap_Kailh_MX_Plated_1.00u
- SW21: renamed from SW20; footprint Button_Switch_Keyboard:SW_Cherry_MX_1.00u_PCB -> PCM_Switch_Keyboard_Hotswap_Kailh:SW_Hotswap_Kailh_MX_Plated_1.00u
- SW22: renamed from SW21; footprint Button_Switch_Keyboard:SW_Cherry_MX_1.00u_PCB -> PCM_Switch_Keyboard_Hotswap_Kailh:SW_Hotswap_Kailh_MX_Plated_1.00u
- SW23: renamed from SW22; footprint Button_Switch_Keyboard:SW_Cherry_MX_1.00u_PCB -> PCM_Switch_Keyboard_Hotswap_Kailh:SW_Hotswap_Kailh_MX_Plated_1.00u
- SW24: renamed from SW23; footprint Button_Switch_Keyboard:SW_Cherry_MX_1.00u_PCB -> PCM_Switch_Keyboard_Hotswap_Kailh:SW_Hotswap_Kailh_MX_Plated_1.00u
- SW25: renamed from SW24; footprint Button_Switch_Keyboard:SW_Cherry_MX_1.00u_PCB -> PCM_Switch_Keyboard_Hotswap_Kailh:SW_Hotswap_Kailh_MX_Plated_1.00u
- SW26: renamed from SW25; footprint Button_Switch_Keyboard:SW_Cherry_MX_1.00u_PCB -> PCM_Switch_Keyboard_Hotswap_Kailh:SW_Hotswap_Kailh_MX_Plated_1.00u
- SW27: renamed from SW26; footprint Button_Switch_Keyboard:SW_Cherry_MX_1.00u_PCB -> PCM_Switch_Keyboard_Hotswap_Kailh:SW_Hotswap_Kailh_MX_Plated_1.00u
- SW28: renamed from SW27; footprint Button_Switch_Keyboard:SW_Cherry_MX_1.00u_PCB -> PCM_Switch_Keyboard_Hotswap_Kailh:SW_Hotswap_Kailh_MX_Plated_1.00u
- SW29: renamed from SW28; footprint Button_Switch_Keyboard:SW_Cherry_MX_1.00u_PCB -> PCM_Switch_Keyboard_Hotswap_Kailh:SW_Hotswap_Kailh_MX_Plated_1.00u
- SW30: renamed from SW29; footprint Button_Switch_Keyboard:SW_Cherry_MX_1.00u_PCB -> PCM_Switch_Keyboard_Hotswap_Kailh:SW_Hotswap_Kailh_MX_Plated_1.00u
- SW31: renamed from SW30; footprint Button_Switch_Keyboard:SW_Cherry_MX_1.50u_PCB -> PCM_Switch_Keyboard_Hotswap_Kailh:SW_Hotswap_Kailh_MX_Plated_1.50u
- SW32: renamed from SW31; footprint Button_Switch_Keyboard:SW_Cherry_MX_1.00u_PCB -> PCM_Switch_Keyboard_Hotswap_Kailh:SW_Hotswap_Kailh_MX_Plated_1.00u
- SW34: renamed from SW33; footprint Button_Switch_Keyboard:SW_Cherry_MX_1.75u_PCB -> PCM_Switch_Keyboard_Hotswap_Kailh:SW_Hotswap_Kailh_MX_Plated_1.75u
- SW35: renamed from SW34; footprint Button_Switch_Keyboard:SW_Cherry_MX_1.00u_PCB -> PCM_Switch_Keyboard_Hotswap_Kailh:SW_Hotswap_Kailh_MX_Plated_1.00u
- SW36: renamed from SW35; footprint Button_Switch_Keyboard:SW_Cherry_MX_1.00u_PCB -> PCM_Switch_Keyboard_Hotswap_Kailh:SW_Hotswap_Kailh_MX_Plated_1.00u
- SW37: renamed from SW36; footprint Button_Switch_Keyboard:SW_Cherry_MX_1.00u_PCB -> PCM_Switch_Keyboard_Hotswap_Kailh:SW_Hotswap_Kailh_MX_Plated_1.00u
- SW38: renamed from SW37; footprint Button_Switch_Keyboard:SW_Cherry_MX_1.00u_PCB -> PCM_Switch_Keyboard_Hotswap_Kailh:SW_Hotswap_Kailh_MX_Plated_1.00u
- SW39: renamed from SW38; footprint Button_Switch_Keyboard:SW_Cherry_MX_1.00u_PCB -> PCM_Switch_Keyboard_Hotswap_Kailh:SW_Hotswap_Kailh_MX_Plated_1.00u
- SW40: renamed from SW39; footprint Button_Switch_Keyboard:SW_Cherry_MX_1.00u_PCB -> PCM_Switch_Keyboard_Hotswap_Kailh:SW_Hotswap_Kailh_MX_Plated_1.00u
- SW41: renamed from SW40; footprint Button_Switch_Keyboard:SW_Cherry_MX_1.00u_PCB -> PCM_Switch_Keyboard_Hotswap_Kailh:SW_Hotswap_Kailh_MX_Plated_1.00u
- SW42: renamed from SW41; footprint Button_Switch_Keyboard:SW_Cherry_MX_1.00u_PCB -> PCM_Switch_Keyboard_Hotswap_Kailh:SW_Hotswap_Kailh_MX_Plated_1.00u
- SW43: renamed from SW42; footprint Button_Switch_Keyboard:SW_Cherry_MX_1.00u_PCB -> PCM_Switch_Keyboard_Hotswap_Kailh:SW_Hotswap_Kailh_MX_Plated_1.00u
- SW44: renamed from SW43; footprint Button_Switch_Keyboard:SW_Cherry_MX_1.00u_PCB -> PCM_Switch_Keyboard_Hotswap_Kailh:SW_Hotswap_Kailh_MX_Plated_1.00u
- SW45: renamed from SW44; footprint Button_Switch_Keyboard:SW_Cherry_MX_1.00u_PCB -> PCM_Switch_Keyboard_Hotswap_Kailh:SW_Hotswap_Kailh_MX_Plated_1.00u
- SW46: renamed from SW45; footprint Button_Switch_Keyboard:SW_Cherry_MX_2.25u_PCB -> PCM_Switch_Keyboard_Hotswap_Kailh:SW_Hotswap_Kailh_MX_Plated_2.25u
- SW47: renamed from SW16; footprint Button_Switch_Keyboard:SW_Cherry_MX_1.00u_PCB -> PCM_Switch_Keyboard_Hotswap_Kailh:SW_Hotswap_Kailh_MX_Plated_1.00u
- SW49: renamed from SW46; footprint Button_Switch_Keyboard:SW_Cherry_MX_2.25u_PCB -> PCM_Switch_Keyboard_Hotswap_Kailh:SW_Hotswap_Kailh_MX_Plated_2.25u
- SW50: renamed from SW47; footprint Button_Switch_Keyboard:SW_Cherry_MX_1.00u_PCB -> PCM_Switch_Keyboard_Hotswap_Kailh:SW_Hotswap_Kailh_MX_Plated_1.00u
- SW51: renamed from SW48; footprint Button_Switch_Keyboard:SW_Cherry_MX_1.00u_PCB -> PCM_Switch_Keyboard_Hotswap_Kailh:SW_Hotswap_Kailh_MX_Plated_1.00u
- SW52: renamed from SW49; footprint Button_Switch_Keyboard:SW_Cherry_MX_1.00u_PCB -> PCM_Switch_Keyboard_Hotswap_Kailh:SW_Hotswap_Kailh_MX_Plated_1.00u
- SW53: renamed from SW50; footprint Button_Switch_Keyboard:SW_Cherry_MX_1.00u_PCB -> PCM_Switch_Keyboard_Hotswap_Kailh:SW_Hotswap_Kailh_MX_Plated_1.00u
- SW54: renamed from SW51; footprint Button_Switch_Keyboard:SW_Cherry_MX_1.00u_PCB -> PCM_Switch_Keyboard_Hotswap_Kailh:SW_Hotswap_Kailh_MX_Plated_1.00u
- SW55: renamed from SW52; footprint Button_Switch_Keyboard:SW_Cherry_MX_1.00u_PCB -> PCM_Switch_Keyboard_Hotswap_Kailh:SW_Hotswap_Kailh_MX_Plated_1.00u
- SW56: renamed from SW53; footprint Button_Switch_Keyboard:SW_Cherry_MX_1.00u_PCB -> PCM_Switch_Keyboard_Hotswap_Kailh:SW_Hotswap_Kailh_MX_Plated_1.00u
- SW57: renamed from SW54; footprint Button_Switch_Keyboard:SW_Cherry_MX_1.00u_PCB -> PCM_Switch_Keyboard_Hotswap_Kailh:SW_Hotswap_Kailh_MX_Plated_1.00u
- SW58: renamed from SW55; footprint Button_Switch_Keyboard:SW_Cherry_MX_1.00u_PCB -> PCM_Switch_Keyboard_Hotswap_Kailh:SW_Hotswap_Kailh_MX_Plated_1.00u
- SW59: renamed from SW56; footprint Button_Switch_Keyboard:SW_Cherry_MX_1.00u_PCB -> PCM_Switch_Keyboard_Hotswap_Kailh:SW_Hotswap_Kailh_MX_Plated_1.00u
- SW60: renamed from SW57; footprint Button_Switch_Keyboard:SW_Cherry_MX_1.75u_PCB -> PCM_Switch_Keyboard_Hotswap_Kailh:SW_Hotswap_Kailh_MX_Plated_1.75u
- SW61: renamed from SW58; footprint Button_Switch_Keyboard:SW_Cherry_MX_1.00u_PCB -> PCM_Switch_Keyboard_Hotswap_Kailh:SW_Hotswap_Kailh_MX_Plated_1.00u
- SW62: renamed from SW32; footprint Button_Switch_Keyboard:SW_Cherry_MX_1.00u_PCB -> PCM_Switch_Keyboard_Hotswap_Kailh:SW_Hotswap_Kailh_MX_Plated_1.00u
- SW64: renamed from SW59; footprint Button_Switch_Keyboard:SW_Cherry_MX_1.25u_PCB -> PCM_Switch_Keyboard_Hotswap_Kailh:SW_Hotswap_Kailh_MX_Plated_1.25u
- SW65: renamed from SW60; footprint Button_Switch_Keyboard:SW_Cherry_MX_1.25u_PCB -> PCM_Switch_Keyboard_Hotswap_Kailh:SW_Hotswap_Kailh_MX_Plated_1.25u
- SW66: renamed from SW61; footprint Button_Switch_Keyboard:SW_Cherry_MX_1.25u_PCB -> PCM_Switch_Keyboard_Hotswap_Kailh:SW_Hotswap_Kailh_MX_Plated_1.25u
- SW67: renamed from SW62; footprint Button_Switch_Keyboard:SW_Cherry_MX_6.25u_PCB -> PCM_Switch_Keyboard_Hotswap_Kailh:SW_Hotswap_Kailh_MX_Plated_6.25u
- SW68: renamed from SW63; footprint Button_Switch_Keyboard:SW_Cherry_MX_1.00u_PCB -> PCM_Switch_Keyboard_Hotswap_Kailh:SW_Hotswap_Kailh_MX_Plated_1.00u
- SW69: renamed from SW64; footprint Button_Switch_Keyboard:SW_Cherry_MX_1.00u_PCB -> PCM_Switch_Keyboard_Hotswap_Kailh:SW_Hotswap_Kailh_MX_Plated_1.00u
- SW70: renamed from SW65; footprint Button_Switch_Keyboard:SW_Cherry_MX_1.00u_PCB -> PCM_Switch_Keyboard_Hotswap_Kailh:SW_Hotswap_Kailh_MX_Plated_1.00u
- SW71: renamed from SW66; footprint Button_Switch_Keyboard:SW_Cherry_MX_1.00u_PCB -> PCM_Switch_Keyboard_Hotswap_Kailh:SW_Hotswap_Kailh_MX_Plated_1.00u
- SW72: renamed from SW67; footprint Button_Switch_Keyboard:SW_Cherry_MX_1.00u_PCB -> PCM_Switch_Keyboard_Hotswap_Kailh:SW_Hotswap_Kailh_MX_Plated_1.00u
- SW73: renamed from SW68; footprint Button_Switch_Keyboard:SW_Cherry_MX_1.00u_PCB -> PCM_Switch_Keyboard_Hotswap_Kailh:SW_Hotswap_Kailh_MX_Plated_1.00u
- renumbered D7 to D10, D6 to D11, D5 to D12, D4 to D13, D3 to D14, D2 to D15, D1 to D16, D31 to D17, D30 to D18, D29 to D19, D15 to D2, D28 to D20, D27 to D21, D26 to D22, D25 to D23, D23 to D25, D22 to D26, D21 to D27, D20 to D28, D19 to D29, D14 to D3, D18 to D30, D17 to D31, D16 to D33, D45 to D34, D44 to D35, D43 to D36, D42 to D37, D41 to D38, D40 to D39, D13 to D4, D39 to D40, D38 to D41, D37 to D42, D36 to D43, D35 to D44, D34 to D45, D33 to D46, D32 to D48, D58 to D49, D12 to D5, D57 to D50, D56 to D51, D55 to D52, D54 to D53, D53 to D54, D52 to D55, D51 to D56, D50 to D57, D49 to D58, D48 to D59, D11 to D6, D47 to D60, D46 to D61, D68 to D63, D67 to D64, D66 to D65, D65 to D66, D64 to D67, D63 to D68, D62 to D69, D10 to D7, D61 to D70, D60 to D71, D59 to D72, D9 to D8, D8 to D9, LED16 to LED17, LED17 to LED18, LED18 to LED19, LED19 to LED20, LED20 to LED21, LED21 to LED22, LED22 to LED23, LED23 to LED24, LED24 to LED25, LED25 to LED26, LED26 to LED27, LED27 to LED28, LED28 to LED29, LED29 to LED30, LED30 to LED31, LED31 to LED33, LED32 to LED35, LED33 to LED36, LED34 to LED37, LED35 to LED38, LED36 to LED39, LED37 to LED40, LED38 to LED41, LED39 to LED42, LED40 to LED43, LED41 to LED44, LED42 to LED45, LED43 to LED46, LED44 to LED48, LED45 to LED49, LED46 to LED50, LED47 to LED51, LED54 to LED53, LED55 to LED54, LED56 to LED55, LED48 to LED56, LED49 to LED57, LED50 to LED58, LED51 to LED59, LED53 to LED60, LED57 to LED61, LED60 to LED62, LED59 to LED64, LED61 to LED65, LED62 to LED66, LED63 to LED67, LED64 to LED68, LED65 to LED69, LED66 to LED70, LED67 to LED71, LED68 to LED72, U2 to U1
Connections:
- net +5V: now also C1.1, C10.2, C11.2, C12.2, C13.2, C14.2, C15.2, C16.2, C17.2, C18.2, C19.2, C2.1, C20.2, C21.2, C22.2, C23.2, C24.2, C25.2, C26.2, C27.2, C28.2, C29.2, C30.2, C31.2, C32.2, C33.2, C34.2, C35.2, C36.2, C37.2, C38.2, C39.2, C40.2, C41.2, C42.2, C43.2, C44.2, C45.2, C46.2, C47.2, C48.2, C49.2, C5.2, C50.2, C51.2, C52.2, C53.2, C54.2, C55.2, C56.2, C57.2, C58.2, C59.2, C6.2, C60.2, C61.2, C62.2, C63.2, C64.2, C65.2, C66.2, C67.2, C68.2, C69.2, C7.2, C70.2, C71.2, C72.2, C73.2, C74.2, C75.2, C76.2, C8.2, C9.2, LED16.1 (VDD), LED32.1 (VDD), LED34.1 (VDD), LED47.1 (VDD), LED63.1 (VDD), R5.1; no longer J1.A4 (VBUS), J1.A9 (VBUS__1), J1.B4 (VBUS__2), J1.B9 (VBUS__3), U1.34 (VCC)
- net GND: now also C1.2, C10.1, C11.1, C12.1, C13.1, C14.1, C15.1, C16.1, C17.1, C18.1, C19.1, C2.2, C20.1, C21.1, C22.1, C23.1, C24.1, C25.1, C26.1, C27.1, C28.1, C29.1, C3.2, C30.1, C31.1, C32.1, C33.1, C34.1, C35.1, C36.1, C37.1, C38.1, C39.1, C4.2, C40.1, C41.1, C42.1, C43.1, C44.1, C45.1, C46.1, C47.1, C48.1, C49.1, C5.1, C51.1, C52.1, C53.1, C54.1, C55.1, C56.1, C57.1, C58.1, C59.1, C6.1, C60.1, C61.1, C62.1, C63.1, C64.1, C65.1, C66.1, C67.1, C68.1, C69.1, C7.1, C70.1, C71.1, C72.1, C73.1, C74.1, C75.1, C76.1, C8.1, C9.1, LED16.3 (GND), LED32.3 (GND), LED34.3 (GND), LED47.3 (GND), LED63.3 (GND), R3.2, R4.2; no longer U1.35 (GND), U1.43 (GND)
- net LED_row3: now also LED61.4 (DIN)
- net col0: now also SW16.S2, SW17.1, SW33.1, SW48.1, SW63.1; no longer SW1.1, SW18.1, SW34.1, SW49.1, SW64.1
- net col10: now also SW26.1, SW42.1, SW56.1, SW9.1; no longer SW10.1, SW27.1, SW43.1, SW57.1
- net col11: now also SW10.1, SW27.1, SW43.1, SW57.1; no longer SW11.1, SW28.1, SW44.1, SW58.1, SW68.1
- net col12: now also SW11.1, SW28.1, SW44.1, SW58.1, SW68.1; no longer SW12.1, SW29.1, SW45.1, SW59.1, SW69.1
- net col13: now also SW12.1, SW29.1, SW45.1, SW59.1, SW69.1; no longer SW13.1, SW30.1, SW70.1
- net col14: now also SW13.1, SW30.1, SW70.1; no longer SW14.1, SW31.1, SW46.1, SW60.1, SW71.1
- net col15: now also SW14.1, SW31.1, SW46.1, SW60.1, SW71.1; no longer SW61.1, SW72.1
- net col16: now also SW61.1, SW72.1; no longer SW15.1, SW32.1, SW47.1, SW62.1, SW73.1
- net col2: now also SW1.1, SW18.1, SW34.1, SW49.1, SW64.1; no longer SW19.1, SW2.1, SW35.1, SW65.1
- net col3: now also SW19.1, SW2.1, SW35.1, SW65.1; no longer SW20.1, SW3.1, SW36.1, SW50.1, SW66.1
- net col4: now also SW20.1, SW3.1, SW36.1, SW50.1, SW66.1; no longer SW21.1, SW37.1, SW4.1, SW51.1
- net col5: now also SW21.1, SW37.1, SW4.1, SW51.1; no longer SW22.1, SW38.1, SW5.1, SW52.1
- net col6: now also SW22.1, SW38.1, SW5.1, SW52.1; no longer SW23.1, SW39.1, SW53.1, SW6.1
- net col7: now also SW23.1, SW39.1, SW53.1, SW6.1; no longer SW24.1, SW40.1, SW54.1, SW67.1, SW7.1
- net col8: now also SW24.1, SW40.1, SW54.1, SW67.1, SW7.1; no longer SW25.1, SW41.1, SW55.1, SW8.1
- net col9: now also SW25.1, SW41.1, SW55.1, SW8.1; no longer SW26.1, SW42.1, SW56.1, SW9.1
- net row0: now also D1.1 (K)
- net row1: now also D32.1 (K)
- net row2: now also D47.1 (K)
- net row3: now also D62.1 (K)
- net row4: now also D73.1 (K)
- net at LED35.2 (DOUT): now also LED34.4 (DIN); no longer LED33.4 (DIN)
- net at LED64.2 (DOUT): now also LED63.4 (DIN)
- net at J1.A5 (CC1): now also R3.1
- net at J1.B5 (CC2): now also R4.1
- net at LED45.4 (DIN), LED46.2 (DOUT): now also C50.1
- net at LED48.2 (DOUT): now also LED47.4 (DIN)
- net at LED33.2 (DOUT): now also LED32.4 (DIN)
- net RESET: now reaches U1.13 (*RESET)
- net RESET: now also R5.2
- net at U1.16 (XTAL2): now also C4.1, Y1.2
- net at U1.17 (XTAL1): now also C3.1, Y1.1
- net at LED17.2 (DOUT): now also LED16.4 (DIN)
- new net: D1.2 (A), SW16.S1
- new net: D32.2 (A), SW17.2
- new net: D73.2 (A), SW63.2
- new net: J1.A4 (VBUS), J1.A9 (VBUS__1), J1.B4 (VBUS__2), J1.B9 (VBUS__3)
- new net: D47.2 (A), SW33.2
- new net: LED33.4 (DIN), LED34.2 (DOUT)
- new net: D62.2 (A), SW48.2
- new net col17: SW15.1, SW32.1, SW47.1, SW62.1, SW73.1
- no-connect marks 0 -> 2
Other:
- moved on the sheet: D10, D11, D12, D13, D14, D15, D16, D17, D18, D19, D20, D21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

Commit message: general updates
Parts:
- removed C35, C36, C51, C76: 0.1u, symbol Device:C
- removed D32, D47, D62, D73: 1N4007, Diode_SMD:D_SOD-123, symbol Diode:1N4007
- removed J1: USB-C, Snapeda:USB4085-GF-A_REVB_GCT_USB4085-GF-A_REVB, symbol Snapeda_kicad_sym:USB4085-GF-A_REVB
- removed LED16, LED32, LED47, LED63: 4960, Snapeda:4960_ADA, symbol Snapeda_kicad_sym:4960
- removed SW16: RotaryEncoder_Switch, Rotary_Encoder:RotaryEncoder_Alps_EC11E-Switch_Vertical_H20mm, symbol Device:RotaryEncoder_Switch
- removed SW17, SW33, SW48, SW63: SW_Push, PCM_Switch_Keyboard_Hotswap_Kailh:SW_Hotswap_Kailh_MX_Plated_1.00u, symbol Switch:SW_Push
- added Boot1: SW_Push, symbol Switch:SW_Push
- added C10, C11, C12, C13, C14, C15, C16, C17, C18, C19, C5, C6, C7, C8, C9: 0.1u, Capacitor_SMD:C_0603_1608Metric, symbol Device:C
- added C88: 1u, Capacitor_SMD:C_0603_1608Metric, symbol Device:C
- added D10, D11, D12, D13, D14, D15, D16, D2, D3, D4, D5, D6, D7, D8, D9: 1N4007, Diode_SMD:D_SOD-123, symbol Diode:1N4007
- added F1: 1.5A, Fuse:Fuse_0603_1608Metric, symbol Device:Polyfuse_Small
- added ICSP1: Conn_01x06_Socket, Connector_PinSocket_2.54mm:PinSocket_1x06_P2.54mm_Vertical, symbol Connector:Conn_01x06_Socket
- added J1: 12402054M611A, Snapeda:12402054M611A_AMPHENOL_12402054M611A, symbol Snapeda_kicad_sym:12402054M611A
- added LED1, LED10, LED11, LED12, LED13, LED14, LED15, LED2, LED3, LED4, LED5, LED6, LED7, LED8, LED9: 4960 Neopixel, 4960_ADA:4960_ADA, symbol Snapeda_kicad_sym:4960
- added SW1: RotaryEncoder_Switch, Rotary_Encoder:RotaryEncoder_Alps_EC11E-Switch_Vertical_H20mm, symbol Device:RotaryEncoder_Switch
- added SW10, SW11, SW12, SW13, SW14, SW15, SW16, SW2, SW3, SW4, SW5, SW6, SW7, SW8, SW9: SW_Push, PCM_Switch_Keyboard_Hotswap_Kailh:SW_Hotswap_Kailh_MX_Plated_1.00u, symbol Switch:SW_Push
- C1, C3, C4, C50: footprint (none) -> Capacitor_SMD:C_0603_1608Metric; Package (none) -> 0603 (1608 Metric)
- C2: value 0.1u -> 4.7uF; footprint (none) -> Capacitor_SMD:C_0603_1608Metric; Package (none) -> 0603 (1608 Metric)
- C20: renamed from C19; footprint (none) -> Capacitor_SMD:C_0603_1608Metric; Package (none) -> 0603 (1608 Metric)
- C21: renamed from C18; footprint (none) -> Capacitor_SMD:C_0603_1608Metric; Package (none) -> 0603 (1608 Metric)
- C22: renamed from C17; footprint (none) -> Capacitor_SMD:C_0603_1608Metric; Package (none) -> 0603 (1608 Metric)
- C23: renamed from C16; footprint (none) -> Capacitor_SMD:C_0603_1608Metric; Package (none) -> 0603 (1608 Metric)
- C24: renamed from C15; footprint (none) -> Capacitor_SMD:C_0603_1608Metric; Package (none) -> 0603 (1608 Metric)
- C25: renamed from C14; footprint (none) -> Capacitor_SMD:C_0603_1608Metric; Package (none) -> 0603 (1608 Metric)
- C26: renamed from C13; footprint (none) -> Capacitor_SMD:C_0603_1608Metric; Package (none) -> 0603 (1608 Metric)
- C27: renamed from C12; footprint (none) -> Capacitor_SMD:C_0603_1608Metric; Package (none) -> 0603 (1608 Metric)
- C28: renamed from C11; footprint (none) -> Capacitor_SMD:C_0603_1608Metric; Package (none) -> 0603 (1608 Metric)
- C29: renamed from C10; footprint (none) -> Capacitor_SMD:C_0603_1608Metric; Package (none) -> 0603 (1608 Metric)
- C30: renamed from C9; footprint (none) -> Capacitor_SMD:C_0603_1608Metric; Package (none) -> 0603 (1608 Metric)
- C31: renamed from C8; footprint (none) -> Capacitor_SMD:C_0603_1608Metric; Package (none) -> 0603 (1608 Metric)
- C32: renamed from C7; footprint (none) -> Capacitor_SMD:C_0603_1608Metric; Package (none) -> 0603 (1608 Metric)
- C33: renamed from C6; footprint (none) -> Capacitor_SMD:C_0603_1608Metric; Package (none) -> 0603 (1608 Metric)
- C34: renamed from C5; footprint (none) -> Capacitor_SMD:C_0603_1608Metric; Package (none) -> 0603 (1608 Metric)
- C35: renamed from C34; footprint (none) -> Capacitor_SMD:C_0603_1608Metric; Package (none) -> 0603 (1608 Metric)
- C36: renamed from C33; footprint (none) -> Capacitor_SMD:C_0603_1608Metric; Package (none) -> 0603 (1608 Metric)
- C37: renamed from C32; footprint (none) -> Capacitor_SMD:C_0603_1608Metric; Package (none) -> 0603 (1608 Metric)
- C38: renamed from C31; footprint (none) -> Capacitor_SMD:C_0603_1608Metric; Package (none) -> 0603 (1608 Metric)
- C39: renamed from C24; footprint (none) -> Capacitor_SMD:C_0603_1608Metric; Package (none) -> 0603 (1608 Metric)
- C40: renamed from C30; footprint (none) -> Capacitor_SMD:C_0603_1608Metric; Package (none) -> 0603 (1608 Metric)
- C41: renamed from C29; footprint (none) -> Capacitor_SMD:C_0603_1608Metric; Package (none) -> 0603 (1608 Metric)
- C42: renamed from C28; footprint (none) -> Capacitor_SMD:C_0603_1608Metric; Package (none) -> 0603 (1608 Metric)
- C43: renamed from C27; footprint (none) -> Capacitor_SMD:C_0603_1608Metric; Package (none) -> 0603 (1608 Metric)
- C44: renamed from C26; footprint (none) -> Capacitor_SMD:C_0603_1608Metric; Package (none) -> 0603 (1608 Metric)
- C45: renamed from C25; footprint (none) -> Capacitor_SMD:C_0603_1608Metric; Package (none) -> 0603 (1608 Metric)
- C46: renamed from C23; footprint (none) -> Capacitor_SMD:C_0603_1608Metric; Package (none) -> 0603 (1608 Metric)
- C47: renamed from C22; footprint (none) -> Capacitor_SMD:C_0603_1608Metric; Package (none) -> 0603 (1608 Metric)
- C48: renamed from C21; footprint (none) -> Capacitor_SMD:C_0603_1608Metric; Package (none) -> 0603 (1608 Metric)
- C49: renamed from C20; footprint (none) -> Capacitor_SMD:C_0603_1608Metric; Package (none) -> 0603 (1608 Metric)
- C51: renamed from C49; footprint (none) -> Capacitor_SMD:C_0603_1608Metric; Package (none) -> 0603 (1608 Metric)
- C52: renamed from C48; footprint (none) -> Capacitor_SMD:C_0603_1608Metric; Package (none) -> 0603 (1608 Metric)
- C53: renamed from C47; footprint (none) -> Capacitor_SMD:C_0603_1608Metric; Package (none) -> 0603 (1608 Metric)
- C54: renamed from C46; footprint (none) -> Capacitor_SMD:C_0603_1608Metric; Package (none) -> 0603 (1608 Metric)
- C55: renamed from C45; footprint (none) -> Capacitor_SMD:C_0603_1608Metric; Package (none) -> 0603 (1608 Metric)
- C56: renamed from C44; footprint (none) -> Capacitor_SMD:C_0603_1608Metric; Package (none) -> 0603 (1608 Metric)
- C57: renamed from C43; footprint (none) -> Capacitor_SMD:C_0603_1608Metric; Package (none) -> 0603 (1608 Metric)
- C58: renamed from C42; footprint (none) -> Capacitor_SMD:C_0603_1608Metric; Package (none) -> 0603 (1608 Metric)
- C59: renamed from C41; footprint (none) -> Capacitor_SMD:C_0603_1608Metric; Package (none) -> 0603 (1608 Metric)
- C60: renamed from C40; footprint (none) -> Capacitor_SMD:C_0603_1608Metric; Package (none) -> 0603 (1608 Metric)
- C61: renamed from C39; footprint (none) -> Capacitor_SMD:C_0603_1608Metric; Package (none) -> 0603 (1608 Metric)
- C62: renamed from C38; footprint (none) -> Capacitor_SMD:C_0603_1608Metric; Package (none) -> 0603 (1608 Metric)
- C63: renamed from C37; footprint (none) -> Capacitor_SMD:C_0603_1608Metric; Package (none) -> 0603 (1608 Metric)
- C64: renamed from C65; footprint (none) -> Capacitor_SMD:C_0603_1608Metric; Package (none) -> 0603 (1608 Metric)
- C65: renamed from C64; footprint (none) -> Capacitor_SMD:C_0603_1608Metric; Package (none) -> 0603 (1608 Metric)
- C66: renamed from C63; footprint (none) -> Capacitor_SMD:C_0603_1608Metric; Package (none) -> 0603 (1608 Metric)
- C67: renamed from C62; footprint (none) -> Capacitor_SMD:C_0603_1608Metric; Package (none) -> 0603 (1608 Metric)
- C68: renamed from C61; footprint (none) -> Capacitor_SMD:C_0603_1608Metric; Package (none) -> 0603 (1608 Metric)
- C69: renamed from C60; footprint (none) -> Capacitor_SMD:C_0603_1608Metric; Package (none) -> 0603 (1608 Metric)
- C70: renamed from C59; footprint (none) -> Capacitor_SMD:C_0603_1608Metric; Package (none) -> 0603 (1608 Metric)
- C71: renamed from C58; footprint (none) -> Capacitor_SMD:C_0603_1608Metric; Package (none) -> 0603 (1608 Metric)
- C72: renamed from C57; footprint (none) -> Capacitor_SMD:C_0603_1608Metric; Package (none) -> 0603 (1608 Metric)
- C73: renamed from C56; footprint (none) -> Capacitor_SMD:C_0603_1608Metric; Package (none) -> 0603 (1608 Metric)
- C74: renamed from C55; footprint (none) -> Capacitor_SMD:C_0603_1608Metric; Package (none) -> 0603 (1608 Metric)
- C75: renamed from C54; footprint (none) -> Capacitor_SMD:C_0603_1608Metric; Package (none) -> 0603 (1608 Metric)
- C76: renamed from C53; footprint (none) -> Capacitor_SMD:C_0603_1608Metric; Package (none) -> 0603 (1608 Metric)
- C77: renamed from C52; footprint (none) -> Capacitor_SMD:C_0603_1608Metric; Package (none) -> 0603 (1608 Metric)
- C78: renamed from C75; footprint (none) -> Capacitor_SMD:C_0603_1608Metric; Package (none) -> 0603 (1608 Metric)
- C79: renamed from C74; footprint (none) -> Capacitor_SMD:C_0603_1608Metric; Package (none) -> 0603 (1608 Metric)
- C80: renamed from C73; footprint (none) -> Capacitor_SMD:C_0603_1608Metric; Package (none) -> 0603 (1608 Metric)
- C81: renamed from C72; footprint (none) -> Capacitor_SMD:C_0603_1608Metric; Package (none) -> 0603 (1608 Metric)
- C82: renamed from C71; footprint (none) -> Capacitor_SMD:C_0603_1608Metric; Package (none) -> 0603 (1608 Metric)
- C83: renamed from C70; footprint (none) -> Capacitor_SMD:C_0603_1608Metric; Package (none) -> 0603 (1608 Metric)
- C84: renamed from C69; footprint (none) -> Capacitor_SMD:C_0603_1608Metric; Package (none) -> 0603 (1608 Metric)
- C85: renamed from C68; footprint (none) -> Capacitor_SMD:C_0603_1608Metric; Package (none) -> 0603 (1608 Metric)
- C86: renamed from C67; footprint (none) -> Capacitor_SMD:C_0603_1608Metric; Package (none) -> 0603 (1608 Metric)
- C87: renamed from C66; footprint (none) -> Capacitor_SMD:C_0603_1608Metric; Package (none) -> 0603 (1608 Metric)
- D1, D61: Package (none) -> SOD-123
- D17: renamed from D16; Package (none) -> SOD-123
- D18: renamed from D15; Package (none) -> SOD-123
- D19: renamed from D14; Package (none) -> SOD-123
- D20: renamed from D13; Package (none) -> SOD-123
- D21: renamed from D12; Package (none) -> SOD-123
- D22: renamed from D11; Package (none) -> SOD-123
- D23: renamed from D10; Package (none) -> SOD-123
- D24: renamed from D9; Package (none) -> SOD-123
- D25: renamed from D8; Package (none) -> SOD-123
- D26: renamed from D7; Package (none) -> SOD-123
- D27: renamed from D6; Package (none) -> SOD-123
- D28: renamed from D5; Package (none) -> SOD-123
- D29: renamed from D4; Package (none) -> SOD-123
- D30: renamed from D3; Package (none) -> SOD-123
- D31: renamed from D2; Package (none) -> SOD-123
- D32: renamed from D31; Package (none) -> SOD-123
- D33: renamed from D30; Package (none) -> SOD-123
- D34: renamed from D29; Package (none) -> SOD-123
- D35: renamed from D28; Package (none) -> SOD-123
- D36: renamed from D27; Package (none) -> SOD-123
- D37: renamed from D26; Package (none) -> SOD-123
- D38: renamed from D25; Package (none) -> SOD-123
- D39: renamed from D24; Package (none) -> SOD-123
- D40: renamed from D23; Package (none) -> SOD-123
- D41: renamed from D22; Package (none) -> SOD-123
- D42: renamed from D21; Package (none) -> SOD-123
- D43: renamed from D20; Package (none) -> SOD-123
- D44: renamed from D19; Package (none) -> SOD-123
- D45: renamed from D18; Package (none) -> SOD-123
- D46: renamed from D17; Package (none) -> SOD-123
- D47: renamed from D46; Package (none) -> SOD-123
- D48: renamed from D45; Package (none) -> SOD-123
- D49: renamed from D44; Package (none) -> SOD-123
- D50: renamed from D43; Package (none) -> SOD-123
- D51: renamed from D42; Package (none) -> SOD-123
- D52: renamed from D41; Package (none) -> SOD-123
- D53: renamed from D40; Package (none) -> SOD-123
- D54: renamed from D39; Package (none) -> SOD-123
- D55: renamed from D38; Package (none) -> SOD-123
- D56: renamed from D37; Package (none) -> SOD-123
- D57: renamed from D36; Package (none) -> SOD-123
- D58: renamed from D35; Package (none) -> SOD-123
- D59: renamed from D34; Package (none) -> SOD-123
- D60: renamed from D33; Package (none) -> SOD-123
- D62: renamed from D60; Package (none) -> SOD-123
- D63: renamed from D59; Package (none) -> SOD-123
- D64: renamed from D58; Package (none) -> SOD-123
- D65: renamed from D57; Package (none) -> SOD-123
- D66: renamed from D56; Package (none) -> SOD-123
- D67: renamed from D55; Package (none) -> SOD-123
- D68: renamed from D54; Package (none) -> SOD-123
- D69: renamed from D53; Package (none) -> SOD-123
- D70: renamed from D52; Package (none) -> SOD-123
- D71: renamed from D51; Package (none) -> SOD-123
- D72: renamed from D50; Package (none) -> SOD-123
- D73: renamed from D49; Package (none) -> SOD-123
- D74: renamed from D48; Package (none) -> SOD-123
- D75: renamed from D72; Package (none) -> SOD-123
- D76: renamed from D71; Package (none) -> SOD-123
- D77: renamed from D70; Package (none) -> SOD-123
- D78: renamed from D69; Package (none) -> SOD-123
- D79: renamed from D68; Package (none) -> SOD-123
- D80: renamed from D67; Package (none) -> SOD-123
- D81: renamed from D66; Package (none) -> SOD-123
- D82: renamed from D65; Package (none) -> SOD-123
- D83: renamed from D64; Package (none) -> SOD-123
- D84: renamed from D63; Package (none) -> SOD-123
- LED16: renamed from LED15; value 4960 -> 4960 Neopixel; footprint Snapeda:4960_ADA -> 4960_ADA:4960_ADA; Package (none) -> 4960
- LED17: renamed from LED14; value 4960 -> 4960 Neopixel; footprint Snapeda:4960_ADA -> 4960_ADA:4960_ADA; Package (none) -> 4960
- LED18: renamed from LED13; value 4960 -> 4960 Neopixel; footprint Snapeda:4960_ADA -> 4960_ADA:4960_ADA; Package (none) -> 4960
- LED19: renamed from LED12; value 4960 -> 4960 Neopixel; footprint Snapeda:4960_ADA -> 4960_ADA:4960_ADA; Package (none) -> 4960
- LED20: renamed from LED11; value 4960 -> 4960 Neopixel; footprint Snapeda:4960_ADA -> 4960_ADA:4960_ADA; Package (none) -> 4960
- LED21: renamed from LED10; value 4960 -> 4960 Neopixel; footprint Snapeda:4960_ADA -> 4960_ADA:4960_ADA; Package (none) -> 4960
- LED22: renamed from LED9; value 4960 -> 4960 Neopixel; footprint Snapeda:4960_ADA -> 4960_ADA:4960_ADA; Package (none) -> 4960
- LED23: renamed from LED8; value 4960 -> 4960 Neopixel; footprint Snapeda:4960_ADA -> 4960_ADA:4960_ADA; Package (none) -> 4960
- LED24: renamed from LED7; value 4960 -> 4960 Neopixel; footprint Snapeda:4960_ADA -> 4960_ADA:4960_ADA; Package (none) -> 4960
- LED25: renamed from LED6; value 4960 -> 4960 Neopixel; footprint Snapeda:4960_ADA -> 4960_ADA:4960_ADA; Package (none) -> 4960
- LED26: renamed from LED5; value 4960 -> 4960 Neopixel; footprint Snapeda:4960_ADA -> 4960_ADA:4960_ADA; Package (none) -> 4960
- LED27: renamed from LED4; value 4960 -> 4960 Neopixel; footprint Snapeda:4960_ADA -> 4960_ADA:4960_ADA; Package (none) -> 4960
- LED28: renamed from LED3; value 4960 -> 4960 Neopixel; footprint Snapeda:4960_ADA -> 4960_ADA:4960_ADA; Package (none) -> 4960
- LED29: renamed from LED2; value 4960 -> 4960 Neopixel; footprint Snapeda:4960_ADA -> 4960_ADA:4960_ADA; Package (none) -> 4960
- LED30: renamed from LED1; value 4960 -> 4960 Neopixel; footprint Snapeda:4960_ADA -> 4960_ADA:4960_ADA; Package (none) -> 4960
- LED31, LED46: value 4960 -> 4960 Neopixel; footprint Snapeda:4960_ADA -> 4960_ADA:4960_ADA; Package (none) -> 4960
- renumbered SW1 to SW17, SW2 to SW18, SW3 to SW19, SW4 to SW20, SW5 to SW21, SW6 to SW22, SW7 to SW23, SW8 to SW24, SW9 to SW25, SW10 to SW26, SW11 to SW27, SW12 to SW28, SW13 to SW29, SW14 to SW30, SW15 to SW31, SW18 to SW32, SW19 to SW33, SW20 to SW34, SW21 to SW35, SW22 to SW36, SW23 to SW37, SW24 to SW38, SW25 to SW39, SW26 to SW40, SW27 to SW41, SW28 to SW42, SW29 to SW43, SW30 to SW44, SW31 to SW45, SW32 to SW46, SW34 to SW47, SW35 to SW48, SW36 to SW49, SW37 to SW50, SW38 to SW51, SW39 to SW52, SW40 to SW53, SW41 to SW54, SW42 to SW55, SW43 to SW56, SW44 to SW57, SW45 to SW58, SW46 to SW59, SW47 to SW60, SW49 to SW61, SW50 to SW62, SW51 to SW63, SW52 to SW64, SW53 to SW65, SW54 to SW66, SW55 to SW67, SW56 to SW68, SW57 to SW69, SW58 to SW70, SW59 to SW71, SW60 to SW72, SW61 to SW73, SW62 to SW74, SW64 to SW75, SW65 to SW76, SW66 to SW77, SW67 to SW78, SW68 to SW79, SW69 to SW80, SW70 to SW81, SW71 to SW82, SW72 to SW83, SW73 to SW84
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Connections:
- net LED_row0 is gone; now on net LED_row1: LED16.4 (DIN)
- net col16 is gone; now on net col14: SW73.1, SW83.1
- net col17 is gone; now on net col15: SW31.1, SW46.1, SW60.1, SW74.1, SW84.1
- net +5V: now also U1.34 (VCC), U1.44 (AVCC), C10.2, C11.2, C12.2, C13.2, C14.2, C15.2, C16.2, C17.2, C18.2, C19.2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; no longer C2.1
- net GND: now also C2.1, C50.1, U1.35 (GND), U1.43 (GND), U1.5 (UGND), Boot1.1, C10.1, C11.1, C12.1, C13.1, C14.1, C15.1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; no longer C2.2
- net LED_row1: now also LED15.2 (DOUT); no longer LED31.4 (DIN)
- net LED_row2: now also LED30.2 (DOUT), LED31.4 (DIN); no longer LED46.4 (DIN)
- net LED_row3: now also LED45.2 (DOUT), LED46.4 (DIN); no longer LED60.4 (DIN)
- net LED_row4: now also LED59.2 (DOUT), LED60.4 (DIN); no longer LED74.4 (DIN)
- net RESET: now also ICSP1.1 (Pin_1)
- net VCC: now also ICSP1.5 (Pin_5)
- net col0: now also SW17.1, SW32.1, SW47.1, SW61.1, SW75.1, U1.33 (PE2), Boot1.2, SW1.S2
- net col10: now also SW27.1, SW42.1, SW57.1, SW70.1, SW79.1, U1.20 (PD2), SW11.1; no longer SW25.1, SW40.1, SW55.1, SW68.1
- net col11: now also SW28.1, SW43.1, SW58.1, SW71.1, SW80.1, U1.21 (PD3), SW12.1; no longer SW26.1, SW41.1, SW56.1, SW69.1
- net col12: now also SW29.1, SW44.1, SW81.1, U1.22 (PD5), SW13.1; no longer SW27.1, SW42.1, SW57.1, SW70.1, SW79.1
- net col13: now also SW30.1, SW45.1, SW59.1, SW72.1, SW82.1, U1.12 (PB7), SW14.1; no longer SW28.1, SW43.1, SW58.1, SW71.1, SW80.1
- net col14: now also U1.8 (PB0), SW15.1; no longer SW29.1, SW44.1, SW81.1
- net col15: now also U1.1 (PE6), SW16.1; no longer SW30.1, SW45.1, SW59.1, SW72.1, SW82.1
- net col2: now also SW19.1, SW34.1, SW49.1, SW62.1, SW77.1, U1.40 (PF1), SW3.1; no longer SW17.1, SW32.1, SW47.1, SW61.1, SW75.1
- net col3: now also SW20.1, SW35.1, SW50.1, SW63.1, U1.39 (PF4), SW4.1; no longer SW18.1, SW33.1, SW48.1, SW76.1
- net col4: now also SW21.1, SW36.1, SW51.1, SW64.1, U1.38 (PF5), SW5.1; no longer SW19.1, SW34.1, SW49.1, SW62.1, SW77.1
- net col5: now also SW22.1, SW37.1, SW52.1, SW65.1, U1.37 (PF6), SW6.1; no longer SW20.1, SW35.1, SW50.1, SW63.1
- net col6: now also SW23.1, SW38.1, SW53.1, SW66.1, SW78.1, U1.36 (PF7), SW7.1; no longer SW21.1, SW36.1, SW51.1, SW64.1
- net col7: now also SW24.1, SW39.1, SW54.1, SW67.1, U1.32 (PC7), SW8.1; no longer SW22.1, SW37.1, SW52.1, SW65.1
- net col8: now also SW25.1, SW40.1, SW55.1, SW68.1, U1.18 (PD0), SW9.1; no longer SW23.1, SW38.1, SW53.1, SW66.1, SW78.1
- net col9: now also SW26.1, SW41.1, SW56.1, SW69.1, U1.19 (PD1), SW10.1; no longer SW24.1, SW39.1, SW54.1, SW67.1
- net row0: now also U1.25 (PD4), D10.1 (K), D11.1 (K), D12.1 (K), D13.1 (K), D14.1 (K), D15.1 (K), D16.1 (K), D2.1 (K), D3.1 (K), D4.1 (K), D5.1 (K)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; no longer D17.1 (K), D18.1 (K), D19.1 (K), D20.1 (K), D21.1 (K), D22.1 (K), D23.1 (K), D24.1 (K), D25.1 (K), D26.1 (K), D27.1 (K), D28.1 (K)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
Other:
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